File: hardware/clock_face/clock_face.kicad_pcb (KiCad board)
At the start: 2 copper layers, 200 x 80 mm, 57 parts, among them J1 Conn_01x04_Pin, J2 Conn_01x06_Pin, J3 Conn_01x04_Pin, J4 Conn_01x04_Pin, U2 HV5530-PQFP, U3 HV5530-PQFP

Commit message: Tweaking existing gerber files and schematics to comply with new project structure
Parts:
- D1, D2, D3, D4, D5, D6: footprint Nixie_Library:LED_SKC6812RV_5.0x4.8x1.6mm -> Nixie Library:SKC6812RV
- NE1, NE2, NE3, NE4: footprint Nixie_Library:INS-1 -> Nixie Library:INS_1
- NX1, NX2, NX3, NX4, NX5, NX6: footprint Nixie_Library:IN_12A_Socket -> Nixie Library:IN_12A
Routing:
- net GND: vias 204 -> 201
Other:
- board text added: "5V+"
- board text added: "MANUFACTURER NOTE(S): - ENIG Finish - Add tented vias on this board. - Surround the edges of this board with edge plating."
- board text removed: "+5V"
- board text removed: "MANUFACTURER NOTE: - Add tented vias on this board. - Surround the edges of this board with edge plating."
