File: hardware/clock_face/main.kicad_sch (KiCad schematic)
At the start: 50 parts, among them J1 Conn_01x04_Pin, J2 Conn_01x06_Pin, J3 Conn_01x04_Pin, J4 Conn_01x04_Pin, U2 HV5530-PQFP, U3 HV5530-PQFP

Commit message: Tweaking existing gerber files and schematics to comply with new project structure
Parts:
- D1, D2, D3, D4, D5, D6: footprint Nixie_Library:LED_SKC6812RV_5.0x4.8x1.6mm -> Nixie Library:SKC6812RV
- NE1, NE2, NE3, NE4: footprint Nixie_Library:INS-1 -> Nixie_Library:INS_1
- NX1, NX3, NX4, NX5, NX6: footprint Nixie_Library:IN_12A_Socket -> Nixie Library:IN_12A
- NX2: footprint Nixie_Library:IN_12A_Socket -> Nixie_Library:IN_12A
Changed lines of the file:
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@@
 			)
 		)
-		(property "Footprint" "Nixie_Library:LED_SKC6812RV_5.0x4.8x1.6mm"
+		(property "Footprint" "Nixie Library:SKC6812RV"
 			(at 175.26 133.35 0)
 			(effects
@@
 			)
 		)
-		(property "Footprint" "Nixie_Library:LED_SKC6812RV_5.0x4.8x1.6mm"
+		(property "Footprint" "Nixie Library:SKC6812RV"
 			(at 281.94 133.35 0)
 			(effects
@@
 			)
 		)
-		(property "Footprint" "Nixie_Library:LED_SKC6812RV_5.0x4.8x1.6mm"
+		(property "Footprint" "Nixie Library:SKC6812RV"
 			(at 138.43 133.35 0)
 			(effects
@@
 			)
 		)
-		(property "Footprint" "Nixie_Library:INS-1"
+		(property "Footprint" "Nixie_Library:INS_1"
 			(at 312.42 226.06 90)
 			(effects
@@
 			)
 		)
-		(property "Footprint" "Nixie_Library:INS-1"
+		(property "Footprint" "Nixie_Library:INS_1"
 			(at 287.02 226.06 90)
 			(effects
@@
 			)
 		)
-		(property "Footprint" "Nixie_Library:INS-1"
+		(property "Footprint" "Nixie_Library:INS_1"
 			(at 274.32 226.06 90)
 			(effects
@@
 			)
 		)
-		(property "Footprint" "Nixie_Library:LED_SKC6812RV_5.0x4.8x1.6mm"
+		(property "Footprint" "Nixie Library:SKC6812RV"
 			(at 210.82 133.35 0)
 			(effects
@@
 			)
 		)
-		(property "Footprint" "Nixie_Library:IN_12A_Socket"
+		(property "Footprint" "Nixie_Library:IN_12A"
 			(at 107.696 262.636 0)
 			(effects
@@
 			)
 		)
-		(property "Footprint" "Nixie_Library:LED_SKC6812RV_5.0x4.8x1.6mm"
+		(property "Footprint" "Nixie Library:SKC6812RV"
 			(at 246.38 133.35 0)
 			(effects
@@
 			)
 		)
-		(property "Footprint" "Nixie_Library:IN_12A_Socket"
+		(property "Footprint" "Nixie Library:IN_12A"
 			(at 215.646 262.636 0)
 			(effects
@@
 			)
 		)
-		(property "Footprint" "Nixie_Library:INS-1"
+		(property "Footprint" "Nixie_Library:INS_1"
 			(at 299.72 226.06 90)
 			(effects
@@
 			)
 		)
-		(property "Footprint" "Nixie_Library:IN_12A_Socket"
+		(property "Footprint" "Nixie Library:IN_12A"
 			(at 107.696 216.916 0)
 			(effects
@@
 			)
 		)
-		(property "Footprint" "Nixie_Library:IN_12A_Socket"
+		(property "Footprint" "Nixie Library:IN_12A"
 			(at 215.646 215.646 0)
 			(effects
@@
 			)
 		)
-		(property "Footprint" "Nixie_Library:IN_12A_Socket"
+		(property "Footprint" "Nixie Library:IN_12A"
 			(at 161.036 215.646 0)
 			(effects
@@
 			)
 		)
-		(property "Footprint" "Nixie_Library:IN_12A_Socket"
+		(property "Footprint" "Nixie Library:IN_12A"
 			(at 161.036 262.636 0)
 			(effects
@@
 			)
 		)
-		(property "Footprint" "Nixie_Library:LED_SKC6812RV_5.0x4.8x1.6mm"
+		(property "Footprint" "Nixie Library:SKC6812RV"
 			(at 101.6 133.35 0)
 			(effects
