File: hardware/control_board/control_board.kicad_pcb (KiCad board)
At the start: 4 copper layers, 200 x 80 mm, 149 parts, among them J1 USB_C_Receptacle_USB2.0_16P, J2 Conn_ARM_SWD_TagConnect_TC203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, J3 USB_C_Receptacle_USB2.0_16P, J4 Conn_01x08, J5 Conn_01x08, J6 Conn_01x08, J7 Conn_01x08, M3 IRLR3110ZTRPBF, Q1 S8050, Q2 S8050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

Commit message: Tweaking existing gerber files and schematics to comply with new project structure
Parts:
- G3: footprint Graphucs:SidePanelArt -> Graphics:SidePanelArt
